File: noise-synth-card.kicad_sch (KiCad schematic)
At the start: 26 parts, among them M1 imogen-wren-card, Q1 BC558, Q2 BC548, U1 40106, U2 TL074

Commit message: finished v1.0 schematic
Parts:
- added C3: 1u, Capacitor_SMD:C_0805_2012Metric_Pad1.18x1.45mm_HandSolder, symbol 000_Capacitor_Film_Immo:cap_film_0805
- added J1: CVpitch, 000_Connectors_Immo:TerminalBlock_Altech_AK300-2_P5.00mm, symbol 000_Connectors_Immo:Screw_Terminal_01x02
- added J2: FM in, 000_Connectors_Immo:TerminalBlock_Altech_AK300-2_P5.00mm, symbol 000_Connectors_Immo:Screw_Terminal_01x02
- added PT4: 100k, Potentiometer_THT:Potentiometer_Bourns_3296W_Vertical, symbol 000_Resistors_Immo:50k_trimpot_MT
- added PT5: B100k, Potentiometer_THT:Potentiometer_Alpha_RD901F-40-00D_Single_Vertical_CircularHoles, symbol 000_Resistors_Immo:Alpha Pot
- added R10, R15, R16: 20k, Resistor_SMD:R_0805_2012Metric_Pad1.20x1.40mm_HandSolder, symbol 000_Resistors_Immo:Resistor_0805
- added R11, R12, R13: 100k, Resistor_SMD:R_0805_2012Metric_Pad1.20x1.40mm_HandSolder, symbol 000_Resistors_Immo:100k
- added R14: 33k, Resistor_SMD:R_0805_2012Metric_Pad1.20x1.40mm_HandSolder, symbol 000_Resistors_Immo:Resistor_0805
- added R9: 200k, Resistor_SMD:R_0805_2012Metric_Pad1.20x1.40mm_HandSolder, symbol 000_Resistors_Immo:Resistor_0805
- added U3: HEF4093B, symbol 4xxx:HEF4093B
Connections:
- net GND: now also J1.1 (Pin_1), J2.1 (Pin_1), PT4.1, PT4.2, R11.1, R12.1, R14.1
- net at R2.1: now also J1.2 (Pin_2)
- net at D2.2 (A), U2.8: now also R9.2
- net at U1.4: now also C3.1
- net at R3.1: now also J2.2 (Pin_2)
- net at U2.9 (-): now also PT4.3, R9.1
- net at U2.6 (-): now also R13.2, R14.2
- net at U2.7: now also R13.1, R15.1
- net at U2.12 (+): now also PT5.2
- net at U2.13 (-): now also U2.14, R16.1
- new net: C3.2, R10.1, R11.2
- new net MIX_OUT: R16.2
- new net SAW: PT5.1, R15.2
- new net SQUARE: PT5.3, R10.2, R12.2
Other:
- moved on the sheet: C2, R7, R8, U1B, U2A, U2B, U2C, U2D

Commit message: dgfhdh
Other:
- note added: "Trimmer NOT thermistor"
- moved on the sheet: J1, J2, JP2, PT2, PT3, R2, R3, R4, R5, TH2, TH3, TH4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
