File: noise-synth-card.kicad_sch (KiCad schematic)
At the start: 42 parts, among them J1 CVpitch, J2 FM in, J3 PWM in, M1 imogen-wren-card, Q1 BC558, Q2 BC548, U1 TL074, U2 TL074, U3 HEF4093B

Commit message: df
Parts:
- removed PT3: B1M, Potentiometer_THT:Potentiometer_Alpha_RD901F-40-00D_Single_Vertical_CircularHoles, symbol 000_Resistors_Immo:Alpha Pot
- added C1, C3: 100n, 000_Capacitors_Immo:C_0805_2012_HandSolder_kawaii, symbol 000_Capacitor_Film_Immo:100n
- added J4: PowerHeader, TerminalBlock_Phoenix:TerminalBlock_Phoenix_MPT-0,5-4-2.54_1x04_P2.54mm_Horizontal, symbol 000-screw-terminals-immo:pheonix_01x04_screwterminal_2.54mm
- added J5: SawOut, 000-screw-terminals-immo:TerminalBlock_Phoenix_MPT-0,5-2-2.54_1x02_P2.54mm_Horizontal, symbol 000-screw-terminals-immo:Screw_Terminal_01x02_small
- added J6: SquareOut, 000-screw-terminals-immo:TerminalBlock_Phoenix_MPT-0,5-2-2.54_1x02_P2.54mm_Horizontal, symbol 000-screw-terminals-immo:Screw_Terminal_01x02_small
- added PT3: 1M, 000_Resistors_Immo:Potentiometer_Bourns_3296W_Vertical, symbol 000_Resistors_Immo:50k_trimpot_MT
- J1, J2, J3: footprint 000_Connectors_Immo:TerminalBlock_Altech_AK300-2_P5.00mm -> 000-screw-terminals-immo:TerminalBlock_Phoenix_MPT-0,5-2-2.54_1x02_P2.54mm_Horizontal; symbol 000_Connectors_Immo:Screw_Terminal_01x02 -> 000-screw-terminals-immo:Screw_Terminal_01x02_small
- PT1, PT2: value B100k -> 100k; footprint Potentiometer_THT:Potentiometer_Alpha_RD901F-40-00D_Single_Vertical_CircularHoles -> 000_Resistors_Immo:Potentiometer_Alpha_RD901F-40-00D_Single_Vertical_CircularHoles
- PT4: renamed from PT6; footprint Potentiometer_THT:Potentiometer_Bourns_3296W_Vertical -> 000_Resistors_Immo:Potentiometer_Bourns_3296W_Vertical; NAME base-note -> base-tune
- PT5: renamed from PT4; footprint Potentiometer_THT:Potentiometer_Bourns_3296W_Vertical -> 000_Resistors_Immo:Potentiometer_Bourns_3296W_Vertical
- PT6: renamed from PT7; value B100k -> 100k; footprint Potentiometer_THT:Potentiometer_Alpha_RD901F-40-00D_Single_Vertical_CircularHoles -> 000_Resistors_Immo:Potentiometer_Alpha_RD901F-40-00D_Single_Vertical_CircularHoles; NAME Pulse Width -> Pulse-Width
- TH1, TH2, TH3, TH4: footprint (none) -> 000_Resistors_Immo:Resistor_0805_2012_handsolder; symbol 000-thermistor-immo:Thermistor -> 000-thermistor-immo:NTC-thermistor-10k-0805; RSpart (none) -> 202-5368; cost (none) -> £0.149; supplier (none) -> https://uk.rs-online.com/web/p/thermistor-ics/2025368?gb=s
- U1: renamed from U3; footprint (none) -> Package_SO:SOIC-14_3.9x8.7mm_P1.27mm; symbol 4xxx:HEF4093B -> 000_Logic_IC_Immo:MC14093B-quad-AND-schmitt-SMD; RSpart (none) -> 518-9192; cost (none) -> £0.50; supplier (none) -> https://uk.rs-online.com/web/p/logic-gates/5189192?gb=s
- U2: footprint (none) -> Package_SO:SOIC-14_3.9x8.7mm_P1.27mm; symbol Amplifier_Operational:TL074 -> 000-op-amp-immo:TL074; RSpart (none) -> 661-0076; cost (none) -> £0.426; supplier (none) -> https://uk.rs-online.com/web/p/op-amps/6610076?gb=s
- U2: renamed from U1; footprint (none) -> Package_SO:SOIC-14_3.9x8.7mm_P1.27mm; symbol Amplifier_Operational:TL074 -> 000-op-amp-immo:TL074; RSpart (none) -> 661-0076; cost (none) -> £0.426; supplier (none) -> https://uk.rs-online.com/web/p/op-amps/6610076?gb=s
- renumbered C1 to C2, C2 to C4, JP2 to JP1, R11 to R1, R19 to R10, R18 to R11, R7 to R12, R9 to R13, R8 to R15, R13 to R17, R15 to R18, R10 to R19, R12 to R2, R17 to R3, R3 to R4, R2 to R5, R1 to R6, R4 to R7, R5 to R8, R6 to R9
Connections:
- net +12V: now also U1.14 (VCC), U2.4 (V+), C1.1, C3.1, J4.4 (Pin_4)
- net -12V: now also U2.11 (V-), C1.2, J4.1 (Pin_1)
- net GND: now also U1.12, U1.13, U1.5, U1.6, U1.7 (GND), U1.8, U1.9, C3.2, J4.2 (Pin_2), J4.3 (Pin_3), J5.1 (Pin_1), J6.1 (Pin_1)
- net SAW: now also J5.2 (Pin_2)
- net SQUARE: now also J6.2 (Pin_2)
- net at JP1.1 (A), Q1.2 (B), R8.2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: now also PT3.1
- net at JP1.2 (C): now also PT3.2
- net at JP1.3 (B), TH4.2: now also PT3.3
- no-connect marks 0 -> 3
Other:
- moved on the sheet: M1, PT1, PT2, R1, R10, R11, R2, R3, R6, R7, TH1, TH2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

Commit message: Added weird pot footprints
Parts:
- removed JP1: fm-dir, Jumper:SolderJumper-3_P1.3mm_Open_RoundedPad1.0x1.5mm_NumberLabels, symbol 000_Connectors_Immo:Jumper_3_Open3small
- PT1, PT2, PT6: footprint 000_Resistors_Immo:Potentiometer_Alpha_RD901F-40-00D_Single_Vertical_CircularHoles -> 000_Resistors_Immo:Potentiometer_Alpha-reversable
- PT3, PT4, PT5: footprint 000_Resistors_Immo:Potentiometer_Bourns_3296W_Vertical -> 000_Resistors_Immo:Potentiometer_Bourns-reversable-1
Connections:
- net at PT3.1, Q1.2 (B), R8.2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: now also PT3.2
Other:
- moved on the sheet: R6, TH1

Commit message: sdgsdf
Parts:
- removed J4: PowerHeader, TerminalBlock_Phoenix:TerminalBlock_Phoenix_MPT-0,5-4-2.54_1x04_P2.54mm_Horizontal, symbol 000-screw-terminals-immo:pheonix_01x04_screwterminal_2.54mm
- added J4: synth-power-header, 000-screw-terminals-immo:synth-power-termbox-MPT-0,5-4-2.54_1x04_P2.54mm, symbol 000-screw-terminals-immo:synth-power-header
Connections:
- net +12V: now also J4.4 (+12v)
- net -12V: now also J4.1 (-12v)
- net GND: now also J4.2 (gnd), J4.3 (gnd)
Changed lines of the file:
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@@
-    )
-  )
-  (symbol (lib_id "000-screw-terminals-immo:pheonix_01x04_screwterminal_2.54mm") (at 189.23 160.02 180) (unit 1)
-    (in_bom yes) (on_board yes) (dnp no) (fields_autoplaced)
-    (property "Reference" "J4" (at 189.23 149.86 0)
-      (effects (font (size 1.27 1.27)))
-    )
-    (property "Value" "PowerHeader" (at 189.23 152.4 0)
-      (effects (font (size 1.27 1.27)))
-    )
-    (property "Footprint" "TerminalBlock_Phoenix:TerminalBlock_Phoenix_MPT-0,5-4-2.54_1x04_P2.54mm_Horizontal" (at 190.5 146.05 0)
-      (effects (font (size 1.27 1.27)) hide)
-    )
-    (property "Datasheet" "https://uk.farnell.com/wago/236-402/terminal-block-wire-to-brd-2pos/dp/1283526" (at 191.77 140.97 0)
-      (effects (font (size 1.27 1.27)) hide)
-    )
-    (pin "1")
-    (pin "2")
-    (pin "3")
-    (pin "4")
-    (instances
-      (project "noise-synth-card"
-        (path "/dee19240-3c10-4a76-9750-c9e476ab49bd"
-          (reference "J4") (unit 1)
-        )
-      )
     )
   )
@@
         )
       )
+    )
+  )
+  (symbol (lib_id "000-screw-terminals-immo:synth-power-header") (at 189.23 160.02 180) (unit 1)
+    (in_bom yes) (on_board yes) (dnp no) (fields_autoplaced)
+    (property "Reference" "J4" (at 186.055 149.86 0)
+      (effects (font (size 1.27 1.27)))
+    )
+    (property "Value" "synth-power-header" (at 186.055 152.4 0)
+      (effects (font (size 1.27 1.27)))
+    )
+    (property "Footprint" "000-screw-terminals-immo:synth-power-termbox-MPT-0,5-4-2.54_1x04_P2.54mm" (at 190.5 146.05 0)
+      (effects (font (size 1.27 1.27)) hide)
+    )
+    (property "Datasheet" "https://uk.farnell.com/wago/236-402/terminal-block-wire-to-brd-2pos/dp/1283526" (at 191.77 140.97 0)
+      (effects (font (size 1.27 1.27)) hide)
+    )
+    (pin "1")
+    (pin "2")
+    (pin "3")
+    (pin "4")
+    (instances
+      (project "noise-synth-card"
+        (path "/dee19240-3c10-4a76-9750-c9e476ab49bd"
+          (reference "J4") (unit 1)
+        )
+      )

Commit message: rtertert
Parts:
- removed C2: 2n2, 000_Capacitors_Immo:C_0805_2012_HandSolder_kawaii, symbol 000_Capacitor_Film_Immo:100n
- removed C4: 1u, Capacitor_SMD:C_0805_2012Metric_Pad1.18x1.45mm_HandSolder, symbol 000_Capacitor_Film_Immo:cap_film_0805
- removed D1: 1N4148, Diode_THT:D_DO-35_SOD27_P7.62mm_Horizontal, symbol 000_Diodes_Immo:1N4148
- removed J1: CVpitch, 000-screw-terminals-immo:TerminalBlock_Phoenix_MPT-0,5-2-2.54_1x02_P2.54mm_Horizontal, symbol 000-screw-terminals-immo:Screw_Terminal_01x02_small
- removed J2: FM in, 000-screw-terminals-immo:TerminalBlock_Phoenix_MPT-0,5-2-2.54_1x02_P2.54mm_Horizontal, symbol 000-screw-terminals-immo:Screw_Terminal_01x02_small
- removed J3: PWM in, 000-screw-terminals-immo:TerminalBlock_Phoenix_MPT-0,5-2-2.54_1x02_P2.54mm_Horizontal, symbol 000-screw-terminals-immo:Screw_Terminal_01x02_small
- removed J5: SawOut, 000-screw-terminals-immo:TerminalBlock_Phoenix_MPT-0,5-2-2.54_1x02_P2.54mm_Horizontal, symbol 000-screw-terminals-immo:Screw_Terminal_01x02_small
- removed J6: SquareOut, 000-screw-terminals-immo:TerminalBlock_Phoenix_MPT-0,5-2-2.54_1x02_P2.54mm_Horizontal, symbol 000-screw-terminals-immo:Screw_Terminal_01x02_small
- removed PT1, PT2, PT6: 100k, 000_Resistors_Immo:Potentiometer_Alpha-reversable, symbol 000_Resistors_Immo:Alpha Pot
- removed PT3: 1M, 000_Resistors_Immo:Potentiometer_Bourns-reversable-1, symbol 000_Resistors_Immo:50k_trimpot_MT
- removed PT4: 1k, 000_Resistors_Immo:Potentiometer_Bourns-reversable-1, symbol 000_Resistors_Immo:50k_trimpot_MT
- removed PT5: 250k, 000_Resistors_Immo:Potentiometer_Bourns-reversable-1, symbol 000_Resistors_Immo:50k_trimpot_MT
- removed Q1: BC558, Package_TO_SOT_THT:TO-92_Inline, symbol Transistor_BJT:BC558
- removed Q2: BC548, Package_TO_SOT_THT:TO-92_Inline, symbol Transistor_BJT:BC548
- removed R1, R11, R12, R15, R17, R3, R4, R5, R6: 100k, Resistor_SMD:R_0805_2012Metric_Pad1.20x1.40mm_HandSolder, symbol 000_Resistors_Immo:100k
- removed R10, R16: 68k, Resistor_SMD:R_0805_2012Metric_Pad1.20x1.40mm_HandSolder, symbol 000_Resistors_Immo:Resistor_0805
- removed R13: 14k, Resistor_SMD:R_0805_2012Metric_Pad1.20x1.40mm_HandSolder, symbol 000_Resistors_Immo:Resistor_0805
- removed R14: 47k, Resistor_SMD:R_0805_2012Metric_Pad1.20x1.40mm_HandSolder, symbol 000_Resistors_Immo:Resistor_0805
- removed R18, R19: 1k, Resistor_SMD:R_0805_2012Metric_Pad1.20x1.40mm_HandSolder, symbol 000_Resistors_Immo:Resistor_0805
- removed R2: 33k, Resistor_SMD:R_0805_2012Metric_Pad1.20x1.40mm_HandSolder, symbol 000_Resistors_Immo:Resistor_0805
- removed R7, R9: 1M, Resistor_SMD:R_0805_2012Metric_Pad1.20x1.40mm_HandSolder, symbol 000_Resistors_Immo:Resistor_0805
- removed R8: 1k5, Resistor_SMD:R_0805_2012Metric_Pad1.20x1.40mm_HandSolder, symbol 000_Resistors_Immo:Resistor_0805
- removed TH1, TH2, TH3, TH4: 10k, 000_Resistors_Immo:Resistor_0805_2012_handsolder, symbol 000-thermistor-immo:NTC-thermistor-10k-0805
- removed unit 1 of U1
- removed unit 3 of U1
- removed unit 4 of U2
- removed unit 1 of U2
- removed unit 3 of U2
- removed unit 2 of U2
- added C7: 100n, 000_Capacitors_Immo:C_0805_2012_HandSolder_kawaii, symbol 000_Capacitor_Film_Immo:100n
- added U3: TL074, Package_SO:SOIC-14_3.9x8.7mm_P1.27mm, symbol 000-op-amp-immo:TL074
- J4: value synth-power-header -> power
Connections:
- net +12V: now also C7.1, U3.4 (V+)
- net -12V: now also C7.2, U3.11 (V-)
- no-connect marks 3 -> 2
Other:
- added sheet VCO-saw-square-0 (vco-saw-square.kicad_sch)
- added sheet VCO-saw-square-1 (vco-saw-square-1.kicad_sch)
- moved on the sheet: C1, C3, J4, M1, U1B, U1D, U1E, U2E

Commit message: dsvgfsdgds
Parts:
- added C8: 100n, 000_Capacitors_Immo:C_0805_2012_HandSolder_kawaii, symbol 000_Capacitor_Film_Immo:100n
- added D3, D4, D8: Blue, Diode_SMD:D_0805_2012Metric_Pad1.15x1.40mm_HandSolder, symbol 000_Diodes_Immo:LED_0805_Blue
- added D5, D6: Pink, Diode_SMD:D_0805_2012Metric_Pad1.15x1.40mm_HandSolder, symbol 000_Diodes_Immo:LED_0805_Blue
- added D7: green, Diode_SMD:D_0805_2012Metric_Pad1.15x1.40mm_HandSolder, symbol 000_Diodes_Immo:LED_0805_Blue
- added J11: Blend Out, 000-screw-terminals-immo:synth-signal-MPT-0,5-2-2.54_1x02_P2.54mm_Horizontal, symbol 000-screw-terminals-immo:synth-signal-header
- added PT13: 1M, 000_Resistors_Immo:Potentiometer_Alpha-reversable, symbol 000_Resistors_Immo:Alpha Pot
- added R39, R40, R41, R42: 1k, Resistor_SMD:R_0805_2012Metric_Pad1.20x1.40mm_HandSolder, symbol 000_Resistors_Immo:1k
- added U4: TL074, Package_SO:SOIC-14_3.9x8.7mm_P1.27mm, symbol 000-op-amp-immo:TL074
Connections:
- net +12V: now also C8.1, R41.2, U4.4 (V+)
- net -12V: now also C8.2, R42.2, U4.11 (V-)
- net GND: now also D7.2 (A), D8.1 (K), J11.1 (gnd), R39.1, R40.1, U4.12 (+), U4.13 (-)
- new net: D3.1 (K), D4.2 (A), R39.2
- new net: J11.2 (signal), U4.1, U4.2 (-)
- new net: D7.1 (K), R42.1
- new net: D5.1 (K), D6.2 (A), PT13.1, U4.6 (-), U4.7
- new net: D5.2 (A), D6.1 (K), R40.2
- new net: D3.2 (A), D4.1 (K), PT13.3, U4.8, U4.9 (-)
- new net: PT13.2, U4.3 (+)
- new net: D8.2 (A), R41.1
- new net VCO-saw-square-0/VCO_OUT: U4.5 (+)
- new net VCO-saw-square-1/VCO_OUT: U4.10 (+)
- no-connect marks 2 -> 3
Other:
- sheet VCO-saw-square-0 ports: added VCO_OUT; removed none
- sheet VCO-saw-square-1 ports: added VCO_OUT; removed none
- note added: "TEST THIS VALUE TOMORROW"
- moved on the sheet: C1, C3, C7, U1E, U2E, U3E

Commit message: ewrtdergf
Parts:
- removed D3, D4, D8: Blue, Diode_SMD:D_0805_2012Metric_Pad1.15x1.40mm_HandSolder, symbol 000_Diodes_Immo:LED_0805_Blue
- removed D5, D6: Pink, Diode_SMD:D_0805_2012Metric_Pad1.15x1.40mm_HandSolder, symbol 000_Diodes_Immo:LED_0805_Blue
- removed D7: green, Diode_SMD:D_0805_2012Metric_Pad1.15x1.40mm_HandSolder, symbol 000_Diodes_Immo:LED_0805_Blue
- added C9: 100p, 000_Capacitors_Immo:C_0805_2012_HandSolder_kawaii, symbol 000_Capacitor_Film_Immo:100n
- added D3, D4: pink, 000_Diodes_Immo:LED_0805_2012_Kawaii, symbol 000_Diodes_Immo:LED_0805_kawaii
- added D5, D6, D8: blue, 000_Diodes_Immo:LED_0805_2012_Kawaii, symbol 000_Diodes_Immo:LED_0805_kawaii
- added D7: green, 000_Diodes_Immo:LED_0805_2012_Kawaii, symbol 000_Diodes_Immo:LED_0805_kawaii
Connections:
- net +12V: now also C9.2
- net GND: now also C9.1, D7.1 (K), D8.2 (A)
- net VCO-saw-square-0/VCO_OUT: now also D5.2 (A), D6.1 (K)
- net VCO-saw-square-1/VCO_OUT: now also D3.1 (K), D4.2 (A)
- net at R39.2: now also D3.2 (A), D4.1 (K)
- net at R42.1: now also D8.1 (K)
- net at R40.2: now also D5.1 (K), D6.2 (A)
- net at R41.1: now also D7.2 (A)
Other:
- note removed: "TEST THIS VALUE TOMORROW"
- moved on the sheet: C3, U1E, U4B, U4C

Commit message: dfgdrfghdf
Parts:
- added C10, C11, C12: 100n, 000_Capacitors_Immo:C_0805_2012_HandSolder_kawaii, symbol 000_Capacitor_Film_Immo:100n
- M1: footprint 000_Modules_Immo:imogen-wren-card -> 000_Modules_Immo:credit-card-screws
Connections:
- net -12V: now also C10.2, C11.2, C12.2; no longer C1.2, C7.2, C8.2
- net GND: now also C1.2, C7.2, C8.2, C10.1, C11.1, C12.1
Other:
- moved on the sheet: C1, C7, C8, U2E, U3E, U4E

Commit message: layout almost finished
Other:
- moved on the sheet: C1, C7
