File: noise-synth-card.kicad_pcb (KiCad board)
At the start: 2 copper layers, 85.1 x 53.3 mm, 21 parts, among them M1 imogen-wren-card, Q1 BC558, Q2 BC548

Commit message: df
Parts:
- removed D2: 1N4148, Diode_THT:D_DO-35_SOD27_P7.62mm_Horizontal
- removed JP2: fm-dir, Jumper:SolderJumper-3_P1.3mm_Open_RoundedPad1.0x1.5mm_NumberLabels
- added C3: 100n, 000_Capacitors_Immo:C_0805_2012_HandSolder_kawaii, F.Cu at (148.9, 40.0)
- added C4: 1u, Capacitor_SMD:C_0805_2012Metric_Pad1.18x1.45mm_HandSolder, F.Cu at (148.9, 43.0)
- added J1: CVpitch, 000-screw-terminals-immo:TerminalBlock_Phoenix_MPT-0,5-2-2.54_1x02_P2.54mm_Horizontal, F.Cu at (106.7, 59.1)
- added J2: FM in, 000-screw-terminals-immo:TerminalBlock_Phoenix_MPT-0,5-2-2.54_1x02_P2.54mm_Horizontal, F.Cu at (106.7, 66.0)
- added J3: PWM in, 000-screw-terminals-immo:TerminalBlock_Phoenix_MPT-0,5-2-2.54_1x02_P2.54mm_Horizontal, F.Cu at (106.7, 73.0)
- added J4: PowerHeader, TerminalBlock_Phoenix:TerminalBlock_Phoenix_MPT-0,5-4-2.54_1x04_P2.54mm_Horizontal, F.Cu at (139.7, 54.0)
- added J5: SawOut, 000-screw-terminals-immo:TerminalBlock_Phoenix_MPT-0,5-2-2.54_1x02_P2.54mm_Horizontal, F.Cu at (181.6, 62.9)
- added J6: SquareOut, 000-screw-terminals-immo:TerminalBlock_Phoenix_MPT-0,5-2-2.54_1x02_P2.54mm_Horizontal, F.Cu at (181.6, 69.8)
- added JP1: fm-dir, Jumper:SolderJumper-3_P1.3mm_Open_RoundedPad1.0x1.5mm_NumberLabels, F.Cu at (116.8, 61.6)
- added PT5: 250k, 000_Resistors_Immo:Potentiometer_Bourns_3296W_Vertical, F.Cu at (120.0, 74.3)
- added PT6: 100k, 000_Resistors_Immo:Potentiometer_Alpha_RD901F-40-00D_Single_Vertical_CircularHoles, F.Cu at (165.4, 99.6)
- added R10: 68k, Resistor_SMD:R_0805_2012Metric_Pad1.20x1.40mm_HandSolder, F.Cu at (128.2, 18.4)
- added R11: 100k, Resistor_SMD:R_0805_2012Metric_Pad1.20x1.40mm_HandSolder, F.Cu at (128.2, 21.4)
- added R12: 100k, Resistor_SMD:R_0805_2012Metric_Pad1.20x1.40mm_HandSolder, F.Cu at (128.2, 24.3)
- added R13: 14k, Resistor_SMD:R_0805_2012Metric_Pad1.20x1.40mm_HandSolder, F.Cu at (128.2, 27.3)
- added R14: 47k, Resistor_SMD:R_0805_2012Metric_Pad1.20x1.40mm_HandSolder, F.Cu at (128.2, 30.2)
- added R15: 100k, Resistor_SMD:R_0805_2012Metric_Pad1.20x1.40mm_HandSolder, F.Cu at (128.2, 33.2)
- added R16: 68k, Resistor_SMD:R_0805_2012Metric_Pad1.20x1.40mm_HandSolder, F.Cu at (128.2, 36.1)
- added R17: 100k, Resistor_SMD:R_0805_2012Metric_Pad1.20x1.40mm_HandSolder, F.Cu at (133.0, 15.5)
- added R18: 1k, Resistor_SMD:R_0805_2012Metric_Pad1.20x1.40mm_HandSolder, F.Cu at (133.0, 18.4)
- added R19: 1k, Resistor_SMD:R_0805_2012Metric_Pad1.20x1.40mm_HandSolder, F.Cu at (133.0, 21.4)
- added TH1: 10k, 000_Resistors_Immo:Resistor_0805_2012_handsolder, F.Cu at (133.0, 24.3)
- added TH2: 10k, 000_Resistors_Immo:Resistor_0805_2012_handsolder, F.Cu at (133.0, 27.3)
- added TH3: 10k, 000_Resistors_Immo:Resistor_0805_2012_handsolder, F.Cu at (133.0, 30.2)
- added TH4: 10k, 000_Resistors_Immo:Resistor_0805_2012_handsolder, F.Cu at (133.0, 33.2)
- added U1: HEF4093B, Package_SO:SOIC-14_3.9x8.7mm_P1.27mm, F.Cu at (150.7, 19.1)
- added U2: TL074, Package_SO:SOIC-14_3.9x8.7mm_P1.27mm, F.Cu at (159.2, 19.1)
- C1: value 2n2 -> 100n
- C2: value 1u -> 2n2; footprint Capacitor_SMD:C_0805_2012Metric_Pad1.18x1.45mm_HandSolder -> 000_Capacitors_Immo:C_0805_2012_HandSolder_kawaii
- M1: moved to B.Cu
- PT1, PT2: value B100k -> 100k; footprint Potentiometer_THT:Potentiometer_Alpha_RD901F-40-00D_Single_Vertical_CircularHoles -> 000_Resistors_Immo:Potentiometer_Alpha_RD901F-40-00D_Single_Vertical_CircularHoles
- PT3: value B1M -> 1M; footprint Potentiometer_THT:Potentiometer_Alpha_RD901F-40-00D_Single_Vertical_CircularHoles -> 000_Resistors_Immo:Potentiometer_Bourns_3296W_Vertical
- PT4: value 100k -> 1k; footprint Potentiometer_THT:Potentiometer_Bourns_3296W_Vertical -> 000_Resistors_Immo:Potentiometer_Bourns_3296W_Vertical
- R2: value 100k -> 33k
- R4, R6: value 1M -> 100k
- R5: value 1k5 -> 100k
- R7: value 100k -> 1M
- R8: value 100k -> 1k5
- R9: value 200k -> 1M
- moved R9 117.9 mm to (128.2, 15.5)
- moved C1 97.5 mm to (148.9, 34.0)
- moved C2 97.5 mm to (148.9, 37.0)
- moved R2 94.5 mm to (123.5, 18.4)
- moved R3 94.5 mm to (123.5, 21.4)
- moved R7 94.5 mm to (123.5, 33.2)
- moved R8 94.5 mm to (123.5, 36.1)
- moved R1 94.5 mm to (123.5, 15.5)
- moved R4 94.5 mm to (123.5, 24.3)
- moved R5 94.5 mm to (123.5, 27.3)
- moved R6 94.5 mm to (123.5, 30.2)
- moved Q1 94.4 mm to (153.3, 35.7)
- moved Q2 94.4 mm to (153.3, 41.5)
- moved D1 84.7 mm to (136.9, 35.1)
- moved PT3 84.3 mm to (120.0, 67.3)
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Connections:
- C1 pad 1: Net-(D1-K) -> +12V
- C1 pad 2: GND -> -12V
- C2 pad 1: Net-(U2A--) -> Net-(D1-K)
- C2 pad 2: Net-(U2B-+) -> GND
- PT1 pad 1: GND -> Net-(PT1-Pad1)
- PT1 pad 3: -12V -> Net-(PT1-Pad3)
- PT2 pad 3: -12V -> Net-(PT2-Pad3)
- PT3 pad 1: Net-(JP2-B) -> Net-(JP1-A)
- PT3 pad 3: Net-(JP2-A) -> Net-(JP1-B)
- PT4 pad 3: Net-(U2C--) -> Net-(PT4-Pad3)
- Q1 pad 2: Net-(JP2-A) -> Net-(JP1-A)
- R1 pad 1: Net-(PT1-Pad2) -> Net-(PT1-Pad1)
- R1 pad 2: Net-(R1-Pad2) -> +12V
- R2 pad 1: unconnected-(R2-Pad1) -> -12V
- R2 pad 2: Net-(R2-Pad2) -> Net-(PT1-Pad3)
- R3 pad 1: unconnected-(R3-Pad1) -> -12V
- R3 pad 2: Net-(R3-Pad2) -> Net-(PT2-Pad3)
- R4 pad 1: Net-(PT2-Pad2) -> Net-(J2-Pin_2)
- R5 pad 2: Net-(JP2-A) -> Net-(R5-Pad2)
- R6 pad 1: Net-(Q1-E) -> Net-(PT1-Pad2)
- R6 pad 2: GND -> Net-(R6-Pad2)
- R7 pad 1: GND -> Net-(PT2-Pad2)
- R7 pad 2: Net-(U2B-+) -> Net-(R7-Pad2)
- R8 pad 1: GND -> Net-(PT4-Pad3)
- R8 pad 2: Net-(D2-K) -> Net-(JP1-A)
- R9 pad 1: Net-(U2C--) -> Net-(Q1-E)
- R9 pad 2: Net-(D2-A) -> +12V

Commit message: Added weird pot footprints
Parts:
- removed JP1: fm-dir, Jumper:SolderJumper-3_P1.3mm_Open_RoundedPad1.0x1.5mm_NumberLabels
- PT1, PT2, PT6: footprint 000_Resistors_Immo:Potentiometer_Alpha_RD901F-40-00D_Single_Vertical_CircularHoles -> 000_Resistors_Immo:Potentiometer_Alpha-reversable
- PT3, PT4, PT5: footprint 000_Resistors_Immo:Potentiometer_Bourns_3296W_Vertical -> 000_Resistors_Immo:Potentiometer_Bourns-reversable-1
- moved PT1 0.28 mm to (144.1, 99.6)
Connections:
- PT3 pad 1: Net-(JP1-A) -> Net-(Q1-B)
- PT3 pad 2: Net-(JP1-C) -> Net-(Q1-B)
- Q1 pad 2: Net-(JP1-A) -> Net-(Q1-B)
- R8 pad 2: Net-(JP1-A) -> Net-(Q1-B)
- TH1 pad 2: Net-(JP1-A) -> Net-(Q1-B)
- TH2 pad 2: Net-(JP1-A) -> Net-(Q1-B)
- TH3 pad 2: Net-(JP1-A) -> Net-(Q1-B)

Commit message: sdgsdf
Parts:
- J4: value PowerHeader -> synth-power-header; footprint TerminalBlock_Phoenix:TerminalBlock_Phoenix_MPT-0,5-4-2.54_1x04_P2.54mm_Horizontal -> 000-screw-terminals-immo:synth-power-termbox-MPT-0,5-4-2.54_1x04_P2.54mm
- moved J4 8.08 mm to (147.3, 56.6), turned to 180 degrees
