File: noise-synth-card.kicad_pcb (KiCad board)
At the start: 2 copper layers, 85.1 x 53.3 mm, 45 parts, among them J1 CVpitch, J2 FM in, J3 PWM in, J4 synth-power-header, J5 SawOut, J6 SquareOut, M1 imogen-wren-card, Q1 BC558, Q2 BC548, U1 HEF4093B, U2 TL074

Commit message: rtertert
Parts:
- added C5: 2n2, 000_Capacitors_Immo:C_0805_2012_HandSolder_kawaii, F.Cu at (143.7, 155.7)
- added C6: 1u, Capacitor_SMD:C_0805_2012Metric_Pad1.18x1.45mm_HandSolder, F.Cu at (143.7, 158.7)
- added C7: 100n, 000_Capacitors_Immo:C_0805_2012_HandSolder_kawaii, F.Cu at (157.0, 137.5)
- added D2: 1N4148, Diode_THT:D_DO-35_SOD27_P7.62mm_Horizontal, F.Cu at (142.9, 152.4)
- added J10: SawOut, 000-screw-terminals-immo:synth-signal-MPT-0,5-2-2.54_1x02_P2.54mm_Horizontal, F.Cu at (181.0, 87.6)
- added J11: SquareOut, 000-screw-terminals-immo:synth-signal-MPT-0,5-2-2.54_1x02_P2.54mm_Horizontal, F.Cu at (181.0, 94.0)
- added J7: CVpitch, 000-screw-terminals-immo:synth-signal-MPT-0,5-2-2.54_1x02_P2.54mm_Horizontal, F.Cu at (107.3, 78.7)
- added J8: FM in, 000-screw-terminals-immo:synth-signal-MPT-0,5-2-2.54_1x02_P2.54mm_Horizontal, F.Cu at (107.3, 85.1)
- added J9: PWM in, 000-screw-terminals-immo:synth-signal-MPT-0,5-2-2.54_1x02_P2.54mm_Horizontal, F.Cu at (107.3, 91.4)
- added PT10: 1k, 000_Resistors_Immo:Potentiometer_Bourns-reversable-1, F.Cu at (116.2, 80.0)
- added PT11: 250k, 000_Resistors_Immo:Potentiometer_Bourns-reversable-1, F.Cu at (116.2, 94.6)
- added PT12: 100k, 000_Resistors_Immo:Potentiometer_Alpha-reversable, F.Cu at (170.7, 89.9)
- added PT7: 100k, 000_Resistors_Immo:Potentiometer_Alpha-reversable, F.Cu at (138.3, 89.9)
- added PT8: 100k, 000_Resistors_Immo:Potentiometer_Alpha-reversable, F.Cu at (154.8, 89.9)
- added PT9: 1M, 000_Resistors_Immo:Potentiometer_Bourns-reversable-1, F.Cu at (116.2, 87.0)
- added Q3: BC558, Package_TO_SOT_THT:TO-92_Inline, F.Cu at (136.8, 153.9)
- added Q4: BC548, Package_TO_SOT_THT:TO-92_Inline, F.Cu at (136.8, 159.7)
- added R20: 100k, Resistor_SMD:R_0805_2012Metric_Pad1.20x1.40mm_HandSolder, F.Cu at (111.8, 152.1)
- added R21: 33k, Resistor_SMD:R_0805_2012Metric_Pad1.20x1.40mm_HandSolder, F.Cu at (111.8, 155.1)
- added R22: 100k, Resistor_SMD:R_0805_2012Metric_Pad1.20x1.40mm_HandSolder, F.Cu at (111.8, 158.0)
- added R23: 100k, Resistor_SMD:R_0805_2012Metric_Pad1.20x1.40mm_HandSolder, F.Cu at (111.8, 160.9)
- added R24: 100k, Resistor_SMD:R_0805_2012Metric_Pad1.20x1.40mm_HandSolder, F.Cu at (111.8, 163.9)
- added R25: 1M, Resistor_SMD:R_0805_2012Metric_Pad1.20x1.40mm_HandSolder, F.Cu at (111.8, 166.8)
- added R26: 100k, Resistor_SMD:R_0805_2012Metric_Pad1.20x1.40mm_HandSolder, F.Cu at (111.8, 169.8)
- added R27: 1k5, Resistor_SMD:R_0805_2012Metric_Pad1.20x1.40mm_HandSolder, F.Cu at (111.8, 172.8)
- added R28: 1M, Resistor_SMD:R_0805_2012Metric_Pad1.20x1.40mm_HandSolder, F.Cu at (116.5, 152.1)
- added R29: 68k, Resistor_SMD:R_0805_2012Metric_Pad1.20x1.40mm_HandSolder, F.Cu at (116.5, 155.1)
- added R30: 100k, Resistor_SMD:R_0805_2012Metric_Pad1.20x1.40mm_HandSolder, F.Cu at (116.5, 158.0)
- added R31: 100k, Resistor_SMD:R_0805_2012Metric_Pad1.20x1.40mm_HandSolder, F.Cu at (116.5, 160.9)
- added R32: 14k, Resistor_SMD:R_0805_2012Metric_Pad1.20x1.40mm_HandSolder, F.Cu at (116.5, 163.9)
- added R33: 47k, Resistor_SMD:R_0805_2012Metric_Pad1.20x1.40mm_HandSolder, F.Cu at (116.5, 166.8)
- added R34: 100k, Resistor_SMD:R_0805_2012Metric_Pad1.20x1.40mm_HandSolder, F.Cu at (116.5, 169.8)
- added R35: 68k, Resistor_SMD:R_0805_2012Metric_Pad1.20x1.40mm_HandSolder, F.Cu at (116.5, 172.8)
- added R36: 100k, Resistor_SMD:R_0805_2012Metric_Pad1.20x1.40mm_HandSolder, F.Cu at (121.3, 152.1)
- added R37: 1k, Resistor_SMD:R_0805_2012Metric_Pad1.20x1.40mm_HandSolder, F.Cu at (121.3, 155.1)
- added R38: 1k, Resistor_SMD:R_0805_2012Metric_Pad1.20x1.40mm_HandSolder, F.Cu at (121.3, 158.0)
- added TH5: 10k, 000_Resistors_Immo:Resistor_0805_2012_handsolder, F.Cu at (121.3, 160.9)
- added TH6: 10k, 000_Resistors_Immo:Resistor_0805_2012_handsolder, F.Cu at (121.3, 163.9)
- added TH7: 10k, 000_Resistors_Immo:Resistor_0805_2012_handsolder, F.Cu at (121.3, 166.8)
- added TH8: 10k, 000_Resistors_Immo:Resistor_0805_2012_handsolder, F.Cu at (121.3, 169.8)
- added U3: TL074, Package_SO:SOIC-14_3.9x8.7mm_P1.27mm, F.Cu at (158.8, 130.9)
- J1, J2, J3, J5, J6: footprint 000-screw-terminals-immo:TerminalBlock_Phoenix_MPT-0,5-2-2.54_1x02_P2.54mm_Horizontal -> 000-screw-terminals-immo:synth-signal-MPT-0,5-2-2.54_1x02_P2.54mm_Horizontal
- J4: value synth-power-header -> power
- R6: value 100k -> 1M
- R7: value 1M -> 100k
- moved U1 56.5 mm to (147.3, 75.5), turned to 90 degrees
- moved PT2 49.9 mm to (154.3, 61.6), turned to 90 degrees
- moved J4 41.0 mm to (181.0, 80.0), turned to 90 degrees
- moved PT1 38.4 mm to (138.4, 61.6), turned to 90 degrees
- moved PT6 38.3 mm to (170.1, 61.6), turned to 90 degrees
- moved PT4 27.3 mm to (116.2, 57.1)
- moved PT3 4.59 mm to (116.2, 64.8), turned to 180 degrees
- moved PT5 4.28 mm to (116.2, 72.4), turned to 180 degrees
- moved J6 3.24 mm to (181.0, 66.7)
- moved J5 2.62 mm to (181.0, 60.3)
- moved J3 2.01 mm to (107.3, 71.1)
- moved J2 1.42 mm to (107.3, 64.8)
- moved J1 0.90 mm to (107.3, 58.4)
Connections:
- net SAW renamed Net-(J5-signal)
- net SQUARE renamed Net-(J6-signal)
- R6 pad 1: Net-(PT1-Pad2) -> Net-(PT2-Pad2)
- R7 pad 1: Net-(PT2-Pad2) -> Net-(PT1-Pad2)
- TH2 pad 1: Net-(R7-Pad2) -> Net-(R5-Pad2)
- TH3 pad 1: Net-(R5-Pad2) -> Net-(R4-Pad2)
- TH3 pad 2: Net-(Q1-B) -> Net-(PT3-Pad3)
- TH4 pad 1: Net-(R4-Pad2) -> Net-(R7-Pad2)
- TH4 pad 2: Net-(PT3-Pad3) -> Net-(Q1-B)
- U1 pad 1: Net-(D1-K) -> Net-(D2-K)
- U1 pad 10: unconnected-(U1-Pad10) -> Net-(D1-A)
- U1 pad 2: Net-(D1-K) -> Net-(D2-K)
- U1 pad 3: Net-(D1-A) -> Net-(D2-A)
- U1 pad 8: GND -> Net-(D1-K)
- U1 pad 9: GND -> Net-(D1-K)

Commit message: dsvgfsdgds
Parts:
- added C8: 100n, 000_Capacitors_Immo:C_0805_2012_HandSolder_kawaii, B.Cu at (168.9, 82.8)
- added D3: Blue, Diode_SMD:D_0805_2012Metric_Pad1.15x1.40mm_HandSolder, F.Cu at (158.1, 67.3)
- added D4: Blue, Diode_SMD:D_0805_2012Metric_Pad1.15x1.40mm_HandSolder, F.Cu at (154.1, 67.3)
- added D5: Pink, Diode_SMD:D_0805_2012Metric_Pad1.15x1.40mm_HandSolder, F.Cu at (158.4, 85.7)
- added D6: Pink, Diode_SMD:D_0805_2012Metric_Pad1.15x1.40mm_HandSolder, F.Cu at (154.1, 85.7)
- added D7: green, Diode_SMD:D_0805_2012Metric_Pad1.15x1.40mm_HandSolder, F.Cu at (172.7, 74.7)
- added D8: Blue, Diode_SMD:D_0805_2012Metric_Pad1.15x1.40mm_HandSolder, F.Cu at (172.7, 66.3)
- added J13: wave-selection, Connector_PinHeader_2.54mm:PinHeader_1x03_P2.54mm_Vertical, F.Cu at (174.6, 52.7)
- added PT13: 1M, 000_Resistors_Immo:Potentiometer_Alpha-reversable, F.Cu at (159.3, 76.6)
- added R39: 1k, Resistor_SMD:R_0805_2012Metric_Pad1.20x1.40mm_HandSolder, F.Cu at (246.0, 49.3)
- added R40: 1k, Resistor_SMD:R_0805_2012Metric_Pad1.20x1.40mm_HandSolder, F.Cu at (246.0, 52.3)
- added R41: 1k, Resistor_SMD:R_0805_2012Metric_Pad1.20x1.40mm_HandSolder, F.Cu at (246.0, 55.2)
- added R42: 1k, Resistor_SMD:R_0805_2012Metric_Pad1.20x1.40mm_HandSolder, F.Cu at (246.0, 58.2)
- added U4: TL074, Package_SO:SOIC-14_3.9x8.7mm_P1.27mm, F.Cu at (168.9, 82.5)
- J10, J5: value SawOut -> VCO-out
- J11: value SquareOut -> Blend Out
- J6: value SquareOut -> wave-selection; footprint 000-screw-terminals-immo:synth-signal-MPT-0,5-2-2.54_1x02_P2.54mm_Horizontal -> Connector_PinHeader_2.54mm:PinHeader_1x03_P2.54mm_Vertical
- moved D2 74.9 mm to (117.5, 81.9)
- moved D1 34.8 mm to (134.6, 69.8), turned to 180 degrees
- moved J6 34.2 mm to (174.6, 100.3), turned to 180 degrees
- moved U1 21.6 mm to (125.7, 76.2)
- moved PT10 20.3 mm to (111.1, 99.7)
- moved J7 12.7 mm to (107.3, 91.4)
- moved J9 12.7 mm to (107.3, 78.7)
- moved J11 9.53 mm to (181.0, 84.5)
- moved PT11 7.65 mm to (115.6, 87.0)
- moved PT5 6.99 mm to (116.2, 65.4)
- moved PT4 6.74 mm to (111.1, 52.7)
- moved PT9 6.38 mm to (115.6, 93.3)
- moved J10 6.35 mm to (181.0, 94.0)
- moved J4 5.72 mm to (181.0, 74.3)
- moved PT3 5.71 mm to (116.2, 59.1)
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Connections:
- J10 pad 2: Net-(J10-signal) -> /VCO-saw-square-1/VCO_OUT
- J5 pad 2: Net-(J5-signal) -> /VCO-saw-square-0/VCO_OUT
- J6 pad 1: GND -> Net-(J6-saw)
- J6 pad 2: Net-(J6-signal) -> /VCO-saw-square-1/VCO_OUT
- R18 pad 2: Net-(J5-signal) -> Net-(J13-saw)
- R19 pad 2: Net-(J6-signal) -> Net-(J13-square)
- R37 pad 2: Net-(J10-signal) -> Net-(J6-saw)
- R38 pad 2: Net-(J11-signal) -> Net-(J6-square)

Commit message: ewrtdergf
Parts:
- removed M1: imogen-wren-card, 000_Modules_Immo:imogen-wren-card
- added C9: 100p, 000_Capacitors_Immo:C_0805_2012_HandSolder_kawaii, B.Cu at (94.6, 75.2)
- added REF**: CreditCard_M3, 000_Modules_Immo:CreditCard_M3, F.Cu at (144.3, 73.4)
- C1, C3, C4, C5, C6, C7, R1, R10, R11, R12, R13, R14, R15, R16, R17, R18, R19, R2, R20, R21, R22, R23, R24, R25, R26, R27, R28, R29, R3, R30, R31, R32, R33, R34, R35, R36, R37, R38, R39, R4, R40, R41, R42, R5, R6, R7, R8, R9, TH1, TH2, TH3, TH4, TH5, TH6, TH7, TH8, U2, U3, U4: moved to B.Cu
- D1, D2: value 1N4148 -> 1N4148_SMD_quatromelf; footprint Diode_THT:D_DO-35_SOD27_P7.62mm_Horizontal -> 000_Diodes_Immo:D_MiniMELF_kawaii
- D3, D4: value Blue -> pink; footprint Diode_SMD:D_0805_2012Metric_Pad1.15x1.40mm_HandSolder -> 000_Diodes_Immo:LED_0805_2012_Kawaii
- D5, D6: value Pink -> blue; footprint Diode_SMD:D_0805_2012Metric_Pad1.15x1.40mm_HandSolder -> 000_Diodes_Immo:LED_0805_2012_Kawaii
- D7: footprint Diode_SMD:D_0805_2012Metric_Pad1.15x1.40mm_HandSolder -> 000_Diodes_Immo:LED_0805_2012_Kawaii
- D8: value Blue -> blue; footprint Diode_SMD:D_0805_2012Metric_Pad1.15x1.40mm_HandSolder -> 000_Diodes_Immo:LED_0805_2012_Kawaii
- J13, J6: value wave-selection -> wave-select; footprint Connector_PinHeader_2.54mm:PinHeader_1x03_P2.54mm_Vertical -> 000_Pin_Headers_Immo:2-way-select
- Q1, Q3: value BC558 -> BC807; footprint Package_TO_SOT_THT:TO-92_Inline -> Package_TO_SOT_SMD:SOT-23; moved to B.Cu
- Q2, Q4: value BC548 -> BC817; footprint Package_TO_SOT_THT:TO-92_Inline -> Package_TO_SOT_SMD:SOT-23; moved to B.Cu
- moved C3 62.1 mm to (97.8, 75.3), turned to -90 degrees
- moved R19 53.9 mm to (138.7, 74.9), turned to 180 degrees
- moved U2 53.2 mm to (142.9, 69.8), turned to -90 degrees
- moved R17 53.1 mm to (149.9, 65.8), turned to 90 degrees
- moved R10 52.0 mm to (117.1, 69.2)
- moved R13 51.0 mm to (146.4, 74.9), turned to 180 degrees
- moved R11 50.8 mm to (164.8, 56.5), turned to 180 degrees
- moved R20 48.9 mm to (160.6, 152.1), turned to 180 degrees
- moved R21 48.9 mm to (160.6, 155.1), turned to 180 degrees
- moved R22 48.9 mm to (160.6, 158.0), turned to 180 degrees
- moved R23 48.9 mm to (160.6, 160.9), turned to 180 degrees
- moved R24 48.9 mm to (160.6, 163.9), turned to 180 degrees
- moved R25 48.9 mm to (160.6, 166.8), turned to 180 degrees
- moved R26 48.9 mm to (160.6, 169.8), turned to 180 degrees
- moved R27 48.9 mm to (160.6, 172.8), turned to 180 degrees
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Connections:
- D3 pad 1: Net-(D3-K) -> /VCO-saw-square-1/VCO_OUT
- D4 pad 2: Net-(D3-K) -> /VCO-saw-square-1/VCO_OUT
- D5 pad 2: Net-(D5-A) -> /VCO-saw-square-0/VCO_OUT
- D6 pad 1: Net-(D5-A) -> /VCO-saw-square-0/VCO_OUT
- D7 pad 1: Net-(D7-K) -> GND
- D7 pad 2: GND -> Net-(D7-A)
- D8 pad 1: GND -> Net-(D8-K)
- D8 pad 2: Net-(D8-A) -> GND
- PT13 pad 1: Net-(D5-K) -> Net-(U4B--)
- PT13 pad 3: Net-(D3-A) -> Net-(U4C--)
- Q1 pad 1: -12V -> Net-(Q1-B)
- Q1 pad 2: Net-(Q1-B) -> Net-(Q1-E)
- Q1 pad 3: Net-(Q1-E) -> -12V
- Q2 pad 1: Net-(D1-K) -> Net-(Q1-E)
- Q2 pad 2: Net-(Q1-E) -> GND
- Q2 pad 3: GND -> Net-(D1-K)
- Q3 pad 1: -12V -> Net-(Q3-B)
- Q3 pad 2: Net-(Q3-B) -> Net-(Q3-E)
- Q3 pad 3: Net-(Q3-E) -> -12V
- Q4 pad 1: Net-(D2-K) -> Net-(Q3-E)
- Q4 pad 2: Net-(Q3-E) -> GND
- Q4 pad 3: GND -> Net-(D2-K)
- R39 pad 2: Net-(D3-K) -> Net-(D3-A)
- R40 pad 2: Net-(D5-A) -> Net-(D5-K)
- R41 pad 1: Net-(D8-A) -> Net-(D7-A)
- R42 pad 1: Net-(D7-K) -> Net-(D8-K)
- U4 pad 6: Net-(D5-K) -> Net-(U4B--)
- U4 pad 7: Net-(D5-K) -> Net-(U4B--)
- U4 pad 8: Net-(D3-A) -> Net-(U4C--)
- U4 pad 9: Net-(D3-A) -> Net-(U4C--)

Commit message: dfgdrfghdf
Parts:
- removed REF**: CreditCard_M3, 000_Modules_Immo:CreditCard_M3
- added C10: 100n, 000_Capacitors_Immo:C_0805_2012_HandSolder_kawaii, B.Cu at (169.9, 88.9)
- added C11: 100n, 000_Capacitors_Immo:C_0805_2012_HandSolder_kawaii, F.Cu at (130.6, 88.3)
- added C12: 100n, 000_Capacitors_Immo:C_0805_2012_HandSolder_kawaii, B.Cu at (145.2, 76.8)
- added M1: imogen-wren-card, 000_Modules_Immo:credit-card-screws, F.Cu at (144.5, 73.3)
- moved R39 93.7 mm to (160.3, 87.0)
- moved R33 89.7 mm to (141.0, 78.4), turned to -90 degrees
- moved R23 89.1 mm to (110.9, 87.0), turned to 0 degrees
- moved R35 88.6 mm to (127.4, 88.9), turned to 0 degrees
- moved TH7 87.2 mm to (110.9, 89.5), turned to 0 degrees
- moved R31 86.7 mm to (131.4, 77.7), turned to -90 degrees
- moved R24 84.3 mm to (110.8, 95.9), turned to 0 degrees
- moved R40 84.3 mm to (163.6, 69.8)
- moved R34 83.7 mm to (134.3, 88.9), turned to 0 degrees
- moved R27 82.1 mm to (119.7, 101.6), turned to 0 degrees
- moved TH6 81.0 mm to (111.8, 93.1), turned to 90 degrees
- moved R37 77.7 mm to (137.8, 78.5), turned to -90 degrees
- moved R32 77.1 mm to (138.2, 88.9)
- moved R36 76.1 mm to (134.6, 77.8), turned to -90 degrees
- moved R26 75.0 mm to (141.0, 97.4), turned to -90 degrees
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Connections:
- C1 pad 2: -12V -> GND
- C7 pad 2: -12V -> GND
- C8 pad 2: -12V -> GND

Commit message: UFKIHGFI
Parts:
- moved C1 24.3 mm to (125.1, 66.9), turned to 90 degrees
- moved C12 21.8 mm to (123.4, 76.2), turned to 0 degrees
- moved C11 19.2 mm to (114.3, 78.1)
- moved C2 16.5 mm to (113.0, 81.7)
- moved C4 15.5 mm to (127.0, 64.2), turned to 90 degrees
- moved R16 15.0 mm to (127.6, 76.5), turned to 90 degrees
- moved R14 13.7 mm to (132.7, 64.3), turned to -90 degrees
- moved R17 13.4 mm to (136.5, 64.5)
- moved J13 12.8 mm to (144.1, 66.7)
- moved R12 12.5 mm to (130.2, 64.3), turned to -90 degrees
- moved U2 11.4 mm to (131.4, 70.4), turned to 0 degrees
- moved R38 11.1 mm to (127.6, 89.9), turned to -90 degrees
- moved R15 11.1 mm to (138.8, 73.7), turned to 0 degrees
- moved R13 8.52 mm to (138.8, 71.1)
- moved R33 7.73 mm to (133.3, 77.1)
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
Commit message: sdfes
Parts:
- moved C5 19.7 mm to (138.9, 82.0), turned to -90 degrees
- moved C2 15.7 mm to (124.2, 70.6), turned to 180 degrees
- moved R18 12.7 mm to (143.5, 53.0), turned to -90 degrees
- moved D5 12.7 mm to (174.2, 57.2)
- moved D6 12.7 mm to (174.2, 61.0), turned to -90 degrees
- moved D3 12.5 mm to (175.0, 94.8), turned to -90 degrees
- moved D4 12.5 mm to (175.0, 90.8)
- moved R17 12.3 mm to (141.0, 53.1)
- moved R16 12.0 mm to (139.4, 74.3), turned to 180 degrees
- moved R21 7.65 mm to (134.3, 101.0)
- moved R14 6.76 mm to (139.4, 63.5), turned to 180 degrees
- moved D1 6.28 mm to (128.0, 76.0), turned to -90 degrees
- moved R13 4.49 mm to (139.4, 66.7)
- moved R15 4.49 mm to (139.4, 69.2)
- moved R12 4.39 mm to (127.6, 60.7)
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Routing:
- net Net-(J9-signal): track 0.00 -> 20.0 mm
- net Net-(J3-signal): track 0.00 -> 17.0 mm
- net Net-(PT5-Pad1): track 0.00 -> 16.6 mm
- net Net-(J11-signal): track 0.00 -> 15.2 mm
- net Net-(PT9-Pad3): track 0.00 -> 13.7 mm
- net Net-(Q3-E): track 0.00 -> 13.1 mm
- net Net-(Q1-B): track 0.00 -> 11.2 mm
- net GND: track 0.00 -> 11.0 mm
- net Net-(PT3-Pad3): track 0.00 -> 9.16 mm
- net Net-(D1-A): track 0.00 -> 8.04 mm
- net Net-(Q3-B): track 0.00 -> 7.92 mm
- net Net-(D1-K): track 0.00 -> 7.54 mm
- net Net-(Q1-E): track 0.00 -> 6.98 mm
- net Net-(PT10-Pad3): track 0.00 -> 6.55 mm
- net Net-(D2-K): track 0.00 -> 4.96 mm
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Other:
- board text added: "+V"

Commit message: layout almost finished
Parts:
- C11, M1: moved to B.Cu
- C5: moved to F.Cu
- moved C8 46.3 mm to (125.2, 85.9), turned to 180 degrees
- moved TH5 29.2 mm to (158.5, 93.2)
- moved C11 26.3 mm to (139.5, 68.3), turned to 180 degrees
- moved C1 24.0 mm to (147.0, 76.2), turned to 180 degrees
- moved R40 20.2 mm to (175.2, 53.3)
- moved U4 19.2 mm to (153.2, 76.2), turned to 0 degrees
- moved R17 19.0 mm to (125.2, 63.8), turned to 180 degrees
- moved R39 18.8 mm to (175.5, 100.3), turned to 180 degrees
- moved C12 18.0 mm to (139.5, 84.3), turned to 180 degrees
- moved D2 17.8 mm to (135.4, 78.9), turned to 90 degrees
- moved C10 16.5 mm to (159.5, 76.2), turned to 180 degrees
- moved R14 15.3 mm to (125.2, 57.9)
- moved R35 14.6 mm to (139.4, 87.1), turned to 180 degrees
- moved TH4 13.7 mm to (142.0, 51.6)
- moved R34 12.7 mm to (132.1, 77.5), turned to 0 degrees
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Routing:
- net GND: track 11.0 -> 484.2 mm, vias 0 -> 18
- net -12V: track 0.00 -> 281.3 mm, vias 0 -> 12
- net +12V: track 0.00 -> 268.9 mm, vias 0 -> 13
- net Net-(U3C--): track 0.00 -> 78.8 mm, vias 0 -> 1
- net Net-(U2C--): track 0.00 -> 63.7 mm, vias 0 -> 2
- net /VCO-saw-square-1/VCO_OUT: track 0.00 -> 59.0 mm, vias 0 -> 1
- net Net-(Q3-B): track 7.92 -> 61.3 mm, vias 0 -> 2
- net Net-(Q1-B): track 11.2 -> 61.2 mm
- net /VCO-saw-square-0/VCO_OUT: track 0.67 -> 50.6 mm, vias 0 -> 1
- net Net-(J11-signal): track 15.2 -> 55.9 mm, vias 0 -> 1
- net Net-(D1-K): track 7.54 -> 42.9 mm, vias 0 -> 2
- net Net-(D2-K): track 4.96 -> 40.0 mm, vias 0 -> 1
- net Net-(U4A-+): track 0.00 -> 26.6 mm, vias 0 -> 1
- net Net-(U4B--): track 0.00 -> 23.0 mm, vias 0 -> 1
- net Net-(U3D-+): track 0.00 -> 21.0 mm, vias 0 -> 1
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- added copper zone on F.Cu, net GND
Other:
- copper layers 2 -> 4

Commit message: sdgdrfgdrfg
Parts:
- moved C5 3.44 mm to (140.6, 80.6), turned to 67.5 degrees
- moved C2 3.34 mm to (117.9, 71.4), turned to -112.5 degrees
- moved D2 3.00 mm to (138.3, 79.8), turned to 67.5 degrees
- moved D1 2.79 mm to (120.7, 72.7), turned to -112.5 degrees
Routing:
- net Net-(D2-K): track 40.0 -> 46.6 mm
- net +12V: track 268.9 -> 264.1 mm
- net Net-(D2-A): track 3.75 -> 7.57 mm
- net Net-(D1-A): track 3.39 -> 7.04 mm
- net Net-(U3C--): track 78.8 -> 77.0 mm, vias 1 -> 3
- net Net-(D1-K): track 42.9 -> 44.2 mm
- net Net-(U3D-+): track 21.0 -> 22.1 mm, vias 1 -> 2
- net Net-(R36-Pad1): track 20.1 -> 21.0 mm, vias 1 -> 2
- net GND: track 484.2 -> 483.3 mm, vias 18 -> 19
