File: noise-synth-card.kicad_pcb (KiCad board)
At the start: 4 copper layers, 85.1 x 53.3 mm, 104 parts, among them J1 CVpitch, J10 VCO-out, J11 Blend Out, J13 wave-select, J2 FM in, J3 PWM in, J4 power, J5 VCO-out, J6 wave-select, J7 CVpitch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

Commit message: dfgdfgd
Connections:
- PT2 pad : (no net) -> GND
Routing:
- net GND: track 483.3 -> 490.0 mm
- net +12V: track 264.1 -> 258.3 mm
- net Net-(D1-K): track 44.2 -> 48.8 mm, vias 2 -> 3

Commit message: dsrfgerge
Parts:
- moved R1 2.92 mm to (142.0, 51.4)
- moved TH4 2.79 mm to (142.0, 54.4)
Connections:
- PT2 pad : GND -> (no net)
Routing:
- net GND: track 490.0 -> 448.3 mm, vias 19 -> 17
- net Net-(J11-signal): track 55.9 -> 35.3 mm, vias 1 -> 2
- net +12V: track 258.3 -> 274.5 mm, vias 13 -> 14
- net Net-(PT7-Pad3): track 3.85 -> 15.8 mm, vias 0 -> 1
- net unconnected-(U1-Pad4): track 2.57 -> 14.2 mm, vias 1 -> 3
- net Net-(PT8-Pad3): track 3.41 -> 13.4 mm, vias 0 -> 1
- net Net-(PT7-Pad1): track 6.26 -> 16.1 mm, vias 0 -> 1
- net Net-(U4C--): track 16.2 -> 25.5 mm
- net Net-(U4B--): track 23.0 -> 32.1 mm, vias 1 -> 2
- net Net-(PT1-Pad1): track 3.60 -> 12.4 mm, vias 0 -> 1
- net Net-(PT1-Pad3): track 3.23 -> 12.0 mm
- net Net-(PT2-Pad3): track 3.44 -> 11.9 mm
- net -12V: track 281.3 -> 288.7 mm, vias 12 -> 14
- net unconnected-(U1-Pad11): track 2.68 -> 9.75 mm
- net Net-(PT4-Pad3): track 3.81 -> 10.2 mm, vias 0 -> 1
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- added copper zone on B.Cu, net GND
Other:
- board text added: "Blend"
- board text added: "Course"
- board text added: "Fine"
- board text added: "Pulse"
- board text added: "Width"

Commit message: sdfsdfs
Other:
- board text added: "Coarse"
- board text removed: "Course"

Commit message: sdfsdfdsf
Parts:
- moved C2 1.30 mm to (116.6, 71.1)
- moved D1 1.03 mm to (119.7, 72.5)
- moved D5 0.78 mm to (175.0, 57.0)
- moved D6 0.77 mm to (175.0, 61.1)
- moved D3 0.75 mm to (175.0, 95.5)
- moved D4 0.52 mm to (175.0, 91.3)
Routing:
- net /VCO-saw-square-0/VCO_OUT: track 51.0 -> 58.3 mm
- net Net-(U4A-+): track 21.4 -> 28.1 mm
- net Net-(J11-signal): track 35.3 -> 39.0 mm
- net Net-(U4B--): track 32.1 -> 35.7 mm
- net GND: track 448.3 -> 451.7 mm
- net Net-(D1-K): track 46.2 -> 49.2 mm
- net Net-(R36-Pad1): track 22.0 -> 20.1 mm
- net /VCO-saw-square-1/VCO_OUT: track 56.9 -> 58.6 mm
- net -12V: track 288.7 -> 290.3 mm
- net Net-(D1-A): track 7.04 -> 8.14 mm
- net +12V: track 274.5 -> 273.6 mm
- net Net-(D3-A): track 12.1 -> 11.6 mm
Other:
- board text added: "Power"
- board text removed: "+V"

Commit message: sdfgdfgd
Parts:
- moved C5 0.96 mm to (140.6, 81.5)
- moved J5 0.76 mm to (181.0, 60.2)
- moved D1 0.62 mm to (119.2, 72.2)
- moved D2 0.55 mm to (138.5, 80.3)
- moved J10 0.51 mm to (181.0, 94.5)
Routing:
- net GND: track 451.7 -> 457.6 mm
- net +12V: track 273.6 -> 278.0 mm
- net /VCO-saw-square-0/VCO_OUT: track 58.3 -> 54.4 mm
- net -12V: track 290.3 -> 292.3 mm
- net Net-(D2-K): track 47.2 -> 48.6 mm
- net /VCO-saw-square-1/VCO_OUT: track 58.6 -> 59.4 mm
- net Net-(D1-A): track 8.14 -> 8.81 mm
- net Net-(D1-K): track 49.2 -> 49.8 mm
- net Net-(PT10-Pad3): track 14.2 -> 14.9 mm

Commit message: sdvsdvsd vs
Parts:
- added G***: LOGO, 000_Graphics_Immo:imogen-wren-5, F.Cu at (178.5, 99.5)
- added G***: LOGO, 000_Graphics_Immo:imogen-wren-10, B.Cu at (169.5, 66.6)
- moved PT9 0.67 mm to (116.2, 93.3)
- moved R3 0.63 mm to (158.5, 58.8)
- moved PT11 0.61 mm to (116.2, 87.0)
- moved R37 0.52 mm to (143.2, 76.2)
- moved R6 0.51 mm to (158.5, 55.9)
- moved TH6 0.37 mm to (112.0, 92.7)
- moved D7 0.36 mm to (179.7, 64.8)
- moved R40 0.34 mm to (174.9, 53.3)
- moved J10 0.13 mm to (181.0, 94.6)
Routing:
- net -12V: track 292.3 -> 302.3 mm
- net +12V: track 278.0 -> 285.4 mm, vias 14 -> 13
- net Net-(Q3-B): track 61.6 -> 66.6 mm, vias 4 -> 3
- net Net-(U3C--): track 77.6 -> 74.7 mm
- net GND: track 457.6 -> 460.2 mm
- net Net-(PT11-Pad1): track 12.8 -> 15.0 mm, vias 1 -> 0
- net Net-(PT9-Pad3): track 13.6 -> 15.5 mm
- net Net-(R36-Pad1): track 20.1 -> 21.4 mm
- net Net-(D5-K): track 11.4 -> 10.4 mm
- net Net-(PT3-Pad3): track 12.1 -> 11.3 mm, vias 2 -> 1
- net Net-(U4B--): track 35.7 -> 36.3 mm
- net Net-(J9-signal): track 17.9 -> 18.5 mm
- net Net-(U3D-+): track 21.4 -> 22.0 mm
- net Net-(J6-saw): track 4.02 -> 4.58 mm
- net Net-(R6-Pad2): track 3.30 -> 2.79 mm
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Other:
- board text added: "Dual VCO"
- board text added: "github.com/ImogenWren"
