File: vco-saw-square.kicad_sch (KiCad schematic)
At the start: 41 parts, among them J1 CVpitch, J2 FM in, J3 PWM in, J5 SawOut, J6 SquareOut, Q1 BC558, Q2 BC548, U1 HEF4093B, U2 TL074

Commit message: dsvgfsdgds
Parts:
- removed J6: SquareOut, 000-screw-terminals-immo:synth-signal-MPT-0,5-2-2.54_1x02_P2.54mm_Horizontal, symbol 000-screw-terminals-immo:synth-signal-header
- added J13: wave-selection, Connector_PinHeader_2.54mm:PinHeader_1x03_P2.54mm_Vertical, symbol 000_Pin_Headers_Immo:2-way-selection
- J5: value SawOut -> VCO-out
Connections:
- net at R19.2: now also J13.3 (square)
- net at R18.2: now also J13.1 (saw); no longer J5.2 (signal)
- new net VCO_OUT: J13.2 (out), J5.2 (signal)
Other:
- moved on the sheet: J5, R18, R19

Commit message: ewrtdergf
Parts:
- removed Q1: BC558, Package_TO_SOT_THT:TO-92_Inline, symbol Transistor_BJT:BC558
- added Q1: BC807, Package_TO_SOT_SMD:SOT-23, symbol 000_Transistors_BJT_Immo:BC807
- D1: value 1N4148 -> 1N4148_SMD_quatromelf; footprint Diode_THT:D_DO-35_SOD27_P7.62mm_Horizontal -> 000_Diodes_Immo:D_MiniMELF_kawaii; symbol 000_Diodes_Immo:1N4148 -> 000_Diodes_Immo:1N4148_SMD_minimelf; RSpart (none) -> 443-3690; cost (none) -> 0.058; supplier (none) -> https://uk.rs-online.com/web/p/switching-diodes/4433690?gb=b
- J13: value wave-selection -> wave-select; footprint Connector_PinHeader_2.54mm:PinHeader_1x03_P2.54mm_Vertical -> 000_Pin_Headers_Immo:2-way-select
- Q2: value BC548 -> BC817; footprint Package_TO_SOT_THT:TO-92_Inline -> Package_TO_SOT_SMD:SOT-23; symbol Transistor_BJT:BC548 -> 000_Transistors_BJT_Immo:BC817; Cost (none) -> £0.082; JLCpart (none) -> C2137; RSpart (none) -> 436-7919; supplier (none) -> https://uk.rs-online.com/web/p/bipolar-transistors/4367919?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
Connections:
- net -12V: now also Q1.3 (C)
- net GND: now also Q2.2 (E); no longer Q2.3 (E)
- net at PT3.1, PT3.2, R8.2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: now also Q1.1 (B)
- net at R9.1: now also Q2.1 (B), Q1.2 (E); no longer Q2.2 (B)
- net at C2.1, D1.1 (K), U1.8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: now also Q2.3 (C); no longer Q2.1 (C)
Changed lines of the file:
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@@
+    )
+  )
+  (symbol (lib_id "000_Transistors_BJT_Immo:BC807") (at 95.25 74.295 0) (mirror x) (unit 1)
+    (in_bom yes) (on_board yes) (dnp no)
+    (property "Reference" "Q1" (at 100.965 76.2 0)
+      (effects (font (size 1.27 1.27)) (justify left))
+    )
+    (property "Value" "BC807" (at 100.965 73.66 0)
+      (effects (font (size 1.27 1.27)) (justify left))
+    )
+    (property "Footprint" "Package_TO_SOT_SMD:SOT-23" (at 91.44 56.515 0)
+      (effects (font (size 1.27 1.27) italic) (justify left) hide)
+    )
+    (property "Datasheet" "https://www.onsemi.com/pub/Collateral/BC808-D.pdf" (at 91.44 53.975 0)
+      (effects (font (size 1.27 1.27)) (justify left) hide)
+    )
+    (property "Sim.Pins" "1=1 2=2 3=3" (at 95.25 74.295 0)
+      (effects (font (size 0 0)) hide)
+    )
+    (property "Sim.Device" "SPICE" (at 100.965 71.12 0)
+      (effects (font (size 1.27 1.27)) (justify left))
+    )
+    (property "Sim.Params" "type=\"X\" model=\"BC807\" lib=\"spice-models\\BC807.lib\"" (at 95.25 74.295 0)
+      (effects (font (size 0 0)) hide)
+    )
+    (property "RSpart" "690-0072" (at 95.25 74.295 0)
+      (effects (font (size 1.27 1.27)) hide)
+    )
+    (property "supplier" "https://uk.rs-online.com/web/p/bipolar-transistors/6900072?gb=s" (at 95.25 74.295 0)
+      (effects (font (size 1.27 1.27)) hide)
+    )
+    (property "cost" "£0.153" (at 95.25 74.295 0)
+      (effects (font (size 1.27 1.27)) hide)
+    )
+    (pin "1")
+    (pin "2")
+    (pin "3")
+    (instances
+      (project "noise-synth-card"
+        (path "/dee19240-3c10-4a76-9750-c9e476ab49bd/b637ddfd-ef78-4820-94bc-7f1d205c735c"
+          (reference "Q1") (unit 1)
+        )
+      )
     )
   )
@@
     )
   )
-  (symbol (lib_id "Transistor_BJT:BC548") (at 118.11 66.675 0) (unit 1)
-    (in_bom yes) (on_board yes) (dnp no) (fields_autoplaced)
-    (property "Reference" "Q2" (at 123.825 66.04 0)
+  (symbol (lib_id "000_Transistors_BJT_Immo:BC817") (at 118.11 66.675 0) (unit 1)
+    (in_bom yes) (on_board yes) (dnp no) (fields_autoplaced)
+    (property "Reference" "Q2" (at 123.19 66.04 0)
       (effects (font (size 1.27 1.27)) (justify left))
     )
-    (property "Value" "BC548" (at 123.825 68.58 0)
+    (property "Value" "BC817" (at 123.19 68.58 0)
       (effects (font (size 1.27 1.27)) (justify left))
     )
-    (property "Footprint" "Package_TO_SOT_THT:TO-92_Inline" (at 123.19 68.58 0)
+    (property "Footprint" "Package_TO_SOT_SMD:SOT-23" (at 130.81 81.28 0)
       (effects (font (size 1.27 1.27) italic) (justify left) hide)
     )
-    (property "Datasheet" "https://www.onsemi.com/pub/Collateral/BC550-D.pdf" (at 118.11 66.675 0)
+    (property "Datasheet" "https://www.onsemi.com/pub/Collateral/BC818-D.pdf" (at 125.73 79.375 0)
       (effects (font (size 1.27 1.27)) (justify left) hide)
+    )
+    (property "Sim.Pins" "1=1 2=2 3=3" (at 118.11 66.675 0)
+      (effects (font (size 0 0)) hide)
+    )
+    (property "Sim.Device" "SPICE" (at 130.81 61.595 0)
+      (effects (font (size 1.27 1.27)) (justify left) hide)
+    )
+    (property "Sim.Params" "type=\"Q\" model=\"BC817\" lib=\"spice-models\\BC817.lib\"" (at 118.11 66.675 0)
+      (effects (font (size 0 0)) hide)
+    )
+    (property "RSpart" "436-7919" (at 118.11 66.675 0)
+      (effects (font (size 1.27 1.27)) hide)
+    )
+    (property "supplier" "https://uk.rs-online.com/web/p/bipolar-transistors/4367919?gb=s" (at 118.11 66.675 0)
+      (effects (font (size 1.27 1.27)) hide)
+    )
+    (property "JLCpart" "C2137" (at 118.11 66.675 0)
+      (effects (font (size 1.27 1.27)) hide)
+    )
+    (property "Cost" "£0.082" (at 118.11 66.675 0)
+      (effects (font (size 1.27 1.27)) hide)
     )
     (pin "1")
@@
     )
   )
-  (symbol (lib_id "Transistor_BJT:BC558") (at 95.25 74.295 0) (mirror x) (unit 1)
-    (in_bom yes) (on_board yes) (dnp no)
-    (property "Reference" "Q1" (at 100.965 74.93 0)
-      (effects (font (size 1.27 1.27)) (justify left))
-    )
-    (property "Value" "BC558" (at 100.965 72.39 0)
-      (effects (font (size 1.27 1.27)) (justify left))
-    )
-    (property "Footprint" "Package_TO_SOT_THT:TO-92_Inline" (at 100.33 72.39 0)
-      (effects (font (size 1.27 1.27) italic) (justify left) hide)
-    )
-    (property "Datasheet" "https://www.onsemi.com/pub/Collateral/BC556BTA-D.pdf" (at 95.25 74.295 0)
-      (effects (font (size 1.27 1.27)) (justify left) hide)
-    )
-    (pin "1")
-    (pin "2")
-    (pin "3")
-    (instances
-      (project "noise-synth-card"
-        (path "/dee19240-3c10-4a76-9750-c9e476ab49bd"
-          (reference "Q1") (unit 1)
-        )
-        (path "/dee19240-3c10-4a76-9750-c9e476ab49bd/b637ddfd-ef78-4820-94bc-7f1d205c735c"
-          (reference "Q1") (unit 1)
-        )
-        (path "/dee19240-3c10-4a76-9750-c9e476ab49bd/0b689d0f-ae27-44dc-b304-30417e2065aa"
-          (reference "Q3") (unit 1)
-        )
-      )
-    )
-  )
   (symbol (lib_id "power:+12V") (at 97.79 53.975 0) (unit 1)
     (in_bom yes) (on_board yes) (dnp no) (fields_autoplaced)
@@
     )
   )
-  (symbol (lib_id "000_Diodes_Immo:1N4148") (at 146.685 46.355 0) (unit 1)
-    (in_bom yes) (on_board yes) (dnp no) (fields_autoplaced)
-    (property "Reference" "D1" (at 146.685 41.275 0)
-      (effects (font (size 1.27 1.27)))
-    )
-    (property "Value" "1N4148" (at 146.685 43.815 0)
-      (effects (font (size 1.27 1.27)))
-    )
-    (property "Footprint" "Diode_THT:D_DO-35_SOD27_P7.62mm_Horizontal" (at 146.685 50.8 0)
-      (effects (font (size 1.27 1.27)) hide)
-    )
-    (property "Datasheet" "https://assets.nexperia.com/documents/data-sheet/1N4148_1N4448.pdf" (at 146.685 46.355 0)
+  (symbol (lib_id "000_Diodes_Immo:1N4148_SMD_minimelf") (at 146.685 46.355 0) (unit 1)
+    (in_bom yes) (on_board yes) (dnp no) (fields_autoplaced)
+    (property "Reference" "D1" (at 146.685 40.64 0)
+      (effects (font (size 1.27 1.27)))
+    )
+    (property "Value" "1N4148_SMD_quatromelf" (at 146.685 43.18 0)
+      (effects (font (size 1.27 1.27)))
+    )
+    (property "Footprint" "000_Diodes_Immo:D_MiniMELF_kawaii" (at 146.685 50.8 0)
+      (effects (font (size 1.27 1.27)) hide)
+    )
+    (property "Datasheet" "https://assets.nexperia.com/documents/data-sheet/1N4148_1N4448.pdf" (at 146.685 48.895 0)
+      (effects (font (size 1.27 1.27)) hide)
+    )
+    (property "RSpart" "443-3690" (at 146.685 46.355 0)
+      (effects (font (size 1.27 1.27)) hide)
+    )
+    (property "supplier" "https://uk.rs-online.com/web/p/switching-diodes/4433690?gb=b" (at 146.685 46.355 0)
+      (effects (font (size 1.27 1.27)) hide)
+    )
+    (property "cost" "0.058" (at 146.685 46.355 0)
       (effects (font (size 1.27 1.27)) hide)
     )
@@
       (effects (font (size 1.27 1.27)) (justify left))
     )
-    (property "Value" "wave-selection" (at 250.825 67.945 0)
+    (property "Value" "wave-select" (at 250.825 67.945 0)
       (effects (font (size 1.27 1.27)) (justify left))
     )
-    (property "Footprint" "Connector_PinHeader_2.54mm:PinHeader_1x03_P2.54mm_Vertical" (at 255.27 61.595 0)
-      (effects (font (size 1.27 1.27)) hide)
-    )
+    (property "Footprint" "000_Pin_Headers_Immo:2-way-select" (at 255.27 61.595 0)
+      (effects (font (size 1.27 1.27)) hide)
+    )
